Commit message: Absolute path commit

File: arm_description/urdf/arm.urdf (robot description, URDF)
Before this commit: robot arm, 17 links, 16 joints
Links:
- link base_link: geometry collision box size=0.09 0.09 0.11; visual mesh filename=file:///home/user/ros2_ws/install/arm_description/share/arm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 scale=0.001 0.001 0.001
- link base_turn: geometry collision mesh filename=file:///home/user/ros2_ws/install/arm_description/share/arm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 scale=0.001 0.001 0.001; visual mesh filename=file:///home/user/ros2_ws/install/arm_description/share/arm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 scale=0.001 0.001 0.001
- link base_turn_rot: geometry collision mesh filename=file:///home/user/ros2_ws/install/arm_description/share/arm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 scale=0.001 0.001 0.001; visual mesh filename=file:///home/user/ros2_ws/install/arm_description/share/arm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 scale=0.001 0.001 0.001
- link crawer_base: geometry collision mesh filename=file:///home/user/ros2_ws/install/arm_description/share/arm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 scale=0.001 0.001 0.001; visual mesh filename=file:///home/user/ros2_ws/install/arm_description/share/arm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 scale=0.001 0.001 0.001
- link crawer_left: geometry collision box size=0.06 0.04 0.04; visual mesh filename=file:///home/user/ros2_ws/install/arm_description/share/arm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 scale=0.001 0.001 0.001
- link crawer_right: geometry collision box size=0.06 0.04 0.04; visual mesh filename=file:///home/user/ros2_ws/install/arm_description/share/arm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 scale=0.001 0.001 0.001
- link dyn2: geometry collision mesh filename=file:///home/user/ros2_ws/install/arm_description/share/arm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 scale=0.01 0.01 0.01; visual mesh filename=file:///home/user/ros2_ws/install/arm_description/share/arm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 scale=0.01 0.01 0.01
- link dyn3: geometry collision mesh filename=file:///home/user/ros2_ws/install/arm_description/share/arm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 scale=0.01 0.01 0.01; visual mesh filename=file:///home/user/ros2_ws/install/arm_description/share/arm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 scale=0.01 0.01 0.01
- link dyn4: geometry collision mesh filename=file:///home/user/ros2_ws/install/arm_description/share/arm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 scale=0.01 0.01 0.01; visual mesh filename=file:///home/user/ros2_ws/install/arm_description/share/arm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 scale=0.01 0.01 0.01
- link dyn5: geometry collision box size=0.05 0.04 0.04; visual mesh filename=file:///home/user/ros2_ws/install/arm_description/share/arm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 scale=0.01 0.01 0.01
- link f4: geometry collision box size=0.05 0.09 0.03; visual mesh filename=file:///home/user/ros2_ws/install/arm_description/share/arm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 scale=0.001 0.001 0.001
- link f5: geometry collision box size=0.05 0.09 0.03; visual mesh filename=file:///home/user/ros2_ws/install/arm_description/share/arm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 scale=0.001 0.001 0.001
- link wrist: geometry collision box size=0.05 0.03 0.04; visual mesh filename=file:///home/user/ros2_ws/install/arm_description/share/arm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 scale=0.001 0.001 0.001
