Commit message: Point 2c

File: arm_description/urdf/arm.urdf.xacro (robot description, xacro)
@@ -1,4 +1,4 @@
 <?xml version="1.0"?>
-<robot name="arm">
+<robot name="arm" xmlns:xacro="http://www.ros.org/wiki/xacro">
   <material name="red">
     <color rgba="1 0 0 1"/>
@@ -7,5 +7,5 @@
     <visual>
       <geometry>
-        <mesh filename="file:///home/user/ros2_ws/install/arm_description/share/arm_description/meshes/base_link.stl" scale="0.001 0.001 0.001"/>
+        <mesh filename="file:///$(find arm_description)/meshes/base_link.stl" scale="0.001 0.001 0.001"/>
       </geometry>
       <origin rpy="0 0 0" xyz="0 0 0"/>
@@ -31,12 +31,12 @@
     <visual>
       <geometry>
-        <mesh filename="file:///home/user/ros2_ws/install/arm_description/share/arm_description/meshes/base_turn.stl" scale="0.001 0.001 0.001"/>
-      </geometry>
-      <origin rpy="0 0 0" xyz="0 0 0"/>
-      <material name="red"/>
-    </visual>
-    <collision>
-      <geometry>
-          <mesh filename="file:///home/user/ros2_ws/install/arm_description/share/arm_description/meshes/base_turn.stl" scale="0.001 0.001 0.001"/>
+        <mesh filename="file:///$(find arm_description)/meshes/base_turn.stl" scale="0.001 0.001 0.001"/>
+      </geometry>
+      <origin rpy="0 0 0" xyz="0 0 0"/>
+      <material name="red"/>
+    </visual>
+    <collision>
+      <geometry>
+          <mesh filename="file:///$(find arm_description)/meshes/base_turn.stl" scale="0.001 0.001 0.001"/>
         </geometry>
       <origin rpy="0 0 0" xyz="0 0 0"/>
@@ -57,11 +57,11 @@
     <visual>
       <geometry>
-        <mesh filename="file:///home/user/ros2_ws/install/arm_description/share/arm_description/meshes/base_turn_table_rot.stl" scale="0.001 0.001 0.001"/>
-      </geometry>
-      <material name="red"/>
-    </visual>
-    <collision>
-      <geometry>
-          <mesh filename="file:///home/user/ros2_ws/install/arm_description/share/arm_description/meshes/base_turn_table_rot.stl" scale="0.001 0.001 0.001"/>
+        <mesh filename="file:///$(find arm_description)/meshes/base_turn_table_rot.stl" scale="0.001 0.001 0.001"/>
+      </geometry>
+      <material name="red"/>
+    </visual>
+    <collision>
+      <geometry>
+          <mesh filename="file:///$(find arm_description)/meshes/base_turn_table_rot.stl" scale="0.001 0.001 0.001"/>
         </geometry>
       <origin rpy="0 0 0" xyz="0 0 0"/>
@@ -80,11 +80,11 @@
     <visual>
       <geometry>
-        <mesh filename="file:///home/user/ros2_ws/install/arm_description/share/arm_description/meshes/dyn.stl" scale="0.01 0.01 0.01"/>
-      </geometry>
-      <origin rpy="0 0 0" xyz="0 0 0"/>
-    </visual>
-    <collision>
-      <geometry>
-          <mesh filename="file:///home/user/ros2_ws/install/arm_description/share/arm_description/meshes/dyn.stl" scale="0.01 0.01 0.01"/>
+        <mesh filename="file:///$(find arm_description)/meshes/dyn.stl" scale="0.01 0.01 0.01"/>
+      </geometry>
+      <origin rpy="0 0 0" xyz="0 0 0"/>
+    </visual>
+    <collision>
+      <geometry>
+          <mesh filename="file:///$(find arm_description)/meshes/dyn.stl" scale="0.01 0.01 0.01"/>
         </geometry>
       <origin rpy="0 0 0" xyz="0 0 0"/>
@@ -112,5 +112,5 @@
     <visual>
       <geometry>
-        <mesh filename="file:///home/user/ros2_ws/install/arm_description/share/arm_description/meshes/f4_n_f3.stl" scale="0.001 0.001 0.001"/>
+        <mesh filename="file:///$(find arm_description)/meshes/f4_n_f3.stl" scale="0.001 0.001 0.001"/>
       </geometry>
       <origin rpy="0 0 0" xyz="0 0 0"/>
@@ -136,11 +136,11 @@
     <visual>
       <geometry>
-        <mesh filename="file:///home/user/ros2_ws/install/arm_description/share/arm_description/meshes/dyn.stl" scale="0.01 0.01 0.01"/>
-      </geometry>
-      <origin rpy="0 0 0" xyz="0 0 0"/>
-    </visual>
-    <collision>
-      <geometry>
-          <mesh filename="file:///home/user/ros2_ws/install/arm_description/share/arm_description/meshes/dyn.stl" scale="0.01 0.01 0.01"/>
+        <mesh filename="file:///$(find arm_description)/meshes/dyn.stl" scale="0.01 0.01 0.01"/>
+      </geometry>
+      <origin rpy="0 0 0" xyz="0 0 0"/>
+    </visual>
+    <collision>
+      <geometry>
+          <mesh filename="file:///$(find arm_description)/meshes/dyn.stl" scale="0.01 0.01 0.01"/>
         </geometry>
       <origin rpy="0 0 0" xyz="0 0 0"/>
@@ -168,5 +168,5 @@
     <visual>
       <geometry>
-        <mesh filename="file:///home/user/ros2_ws/install/arm_description/share/arm_description/meshes/f4_n_f3.stl" scale="0.001 0.001 0.001"/>
+        <mesh filename="file:///$(find arm_description)/meshes/f4_n_f3.stl" scale="0.001 0.001 0.001"/>
       </geometry>
       <origin rpy="0 0 0" xyz="0 0 0"/>
@@ -191,11 +191,11 @@
     <visual>
       <geometry>
-        <mesh filename="file:///home/user/ros2_ws/install/arm_description/share/arm_description/meshes/dyn.stl" scale="0.01 0.01 0.01"/>
-      </geometry>
-      <origin rpy="0 0 0" xyz="0 0 0"/>
-    </visual>
-    <collision>
-      <geometry>
-          <mesh filename="file:///home/user/ros2_ws/install/arm_description/share/arm_description/meshes/dyn.stl" scale="0.01 0.01 0.01"/>
+        <mesh filename="file:///$(find arm_description)/meshes/dyn.stl" scale="0.01 0.01 0.01"/>
+      </geometry>
+      <origin rpy="0 0 0" xyz="0 0 0"/>
+    </visual>
+    <collision>
+      <geometry>
+          <mesh filename="file:///$(find arm_description)/meshes/dyn.stl" scale="0.01 0.01 0.01"/>
         </geometry>
       <origin rpy="0 0 0" xyz="0 0 0"/>
@@ -223,5 +223,5 @@
     <visual>
       <geometry>
-        <mesh filename="file:///home/user/ros2_ws/install/arm_description/share/arm_description/meshes/wrist.stl" scale="0.001 0.001 0.001"/>
+        <mesh filename="file:///$(find arm_description)/meshes/wrist.stl" scale="0.001 0.001 0.001"/>
       </geometry>
       <origin rpy="0 0 0" xyz="0 0 0"/>
@@ -247,5 +247,5 @@
     <visual>
       <geometry>
-        <mesh filename="file:///home/user/ros2_ws/install/arm_description/share/arm_description/meshes/dyn.stl" scale="0.01 0.01 0.01"/>
+        <mesh filename="file:///$(find arm_description)/meshes/dyn.stl" scale="0.01 0.01 0.01"/>
       </geometry>
       <origin rpy="0 0 0" xyz="0 0 0"/>
@@ -279,12 +279,12 @@
     <visual>
       <geometry>
-        <mesh filename="file:///home/user/ros2_ws/install/arm_description/share/arm_description/meshes/the_crawer_base.stl" scale="0.001 0.001 0.001"/>
-      </geometry>
-      <origin rpy="0 0 0" xyz="0 0 0"/>
-      <material name="red"/>
-    </visual>
-    <collision>
-      <geometry>
-          <mesh filename="file:///home/user/ros2_ws/install/arm_description/share/arm_description/meshes/the_crawer_base.stl" scale="0.001 0.001 0.001"/>
+        <mesh filename="file:///$(find arm_description)/meshes/the_crawer_base.stl" scale="0.001 0.001 0.001"/>
+      </geometry>
+      <origin rpy="0 0 0" xyz="0 0 0"/>
+      <material name="red"/>
+    </visual>
+    <collision>
+      <geometry>
+          <mesh filename="file:///$(find arm_description)/meshes/the_crawer_base.stl" scale="0.001 0.001 0.001"/>
         </geometry>
       <origin rpy="0 0 0" xyz="0 0 0"/>
@@ -303,5 +303,5 @@
     <visual>
       <geometry>
-        <mesh filename="file:///home/user/ros2_ws/install/arm_description/share/arm_description/meshes/the_crawer.stl" scale="0.001 0.001 0.001"/>
+        <mesh filename="file:///$(find arm_description)/meshes/the_crawer.stl" scale="0.001 0.001 0.001"/>
       </geometry>
       <origin rpy="0 0 0" xyz="0 0 0"/>
@@ -329,5 +329,5 @@
     <visual>
       <geometry>
-        <mesh filename="file:///home/user/ros2_ws/install/arm_description/share/arm_description/meshes/the_crawer.stl" scale="0.001 0.001 0.001"/>
+        <mesh filename="file:///$(find arm_description)/meshes/the_crawer.stl" scale="0.001 0.001 0.001"/>
       </geometry>
       <origin rpy="0 0 0" xyz="0 0 0"/>

Commit message: Point 2d

File: arm_description/urdf/arm.urdf.xacro (robot description, xacro)
@@ -1,4 +1,5 @@
 <?xml version="1.0"?>
 <robot name="arm" xmlns:xacro="http://www.ros.org/wiki/xacro">
+  <xacro:include filename="file:///$(find arm_description)/urdf/arm_hardware_interface.xacro"/>
   <material name="red">
     <color rgba="1 0 0 1"/>

File: arm_description/urdf/arm_hardware_interface.xacro (robot description, xacro)
@@ -1,21 +1,21 @@
 <?xml version="1.0"?>
-<robot xmlns:xacro="http://www.ros.org/wiki/xacro">
-  <xacro:macro name="define_joint_interface" params="joint_name">
-    <joint name="${joint_name}" type="revolute">
-      <parent link="base_turn"/>
-      <child link="base_turn_rot"/>
-      <origin xyz="-0.0 0.0155 0.013" rpy="0 0 -1.57"/>
-      <axis xyz="0 0 1" />
-      <limit effort="300" velocity="0.1" lower="-2.57" upper="2.57"/>
-      <ros2_control>
-        <hardware_interface>PositionJointInterface</hardware_interface>
+<robot xmlns:xacro="http://www.ros.org/wiki/xacro"
+       xmlns:ros2_control="http://ros2-control.ros.org/">
+  <xacro:macro name="joint_hardware_interface" params="name initial_pos">
+    <joint name="${name}" type="revolute">
+      <ros2_control name="${name}" type="system">
+         <hardware_interface>PositionJointInterface</hardware_interface>
+         <command_interface name="position"/>
+         <state_interface name="position">
+           <param name="initial_value">${initial_pos}</param>
+         </state_interface>
+         <state_interface name="velocity">
+           <param name="initial_value">0.0</param>
+         </state_interface>
+         <state_interface name="effort">
+           <param name="initial_value">0.0</param>
+         </state_interface>
       </ros2_control>
     </joint>
   </xacro:macro>
-  <!-- Use the macro for your joints -->
-  <xacro:define_joint_interface joint_name="j0"/>
-  <xacro:define_joint_interface joint_name="j1"/>
-  <xacro:define_joint_interface joint_name="j2"/>
-  <xacro:define_joint_interface joint_name="j3"/>
-  <!-- Add any other joints as necessary -->
 </robot>

Commit message: Point 2e

File: arm_description/urdf/arm.urdf.xacro (robot description, xacro)
@@ -1,5 +1,5 @@
 <?xml version="1.0"?>
 <robot name="arm" xmlns:xacro="http://www.ros.org/wiki/xacro">
-  <xacro:include filename="file:///$(find arm_description)/urdf/arm_hardware_interface.xacro"/>
+  <xacro:include filename="$(find arm_description)/urdf/arm_hardware_interface.xacro"/>
   <material name="red">
     <color rgba="1 0 0 1"/>
@@ -348,3 +348,18 @@
     </inertial>
   </link>
+    <gazebo>
+    <plugin filename="ign_ros2_control-system" name="ign_ros2_control::IgnitionROS2ControlPlugin">
+    <parameters>$(find arm_description)/config/arm_joint_controller.yaml</parameters>
+      <controller_manager_prefix_node_name>controller_manager</controller_manager_prefix_node_name>
+    </plugin>
+  </gazebo>
+  <ros2_control name="HardwareInterface_Ignition" type="system">
+    <hardware>
+      <plugin>ign_ros2_control/IgnitionSystem</plugin>
+    </hardware>
+    <xacro:arm_hardware_interface name="j0" initial_pos="0.1" />
+    <xacro:arm_hardware_interface name="j1" initial_pos="0.1" />
+    <xacro:arm_hardware_interface name="j2" initial_pos="0.1" />
+    <xacro:arm_hardware_interface name="j3" initial_pos="0.1" />
+  </ros2_control>
 </robot>

File: arm_description/urdf/arm_hardware_interface.xacro (robot description, xacro)
@@ -2,7 +2,6 @@
 <robot xmlns:xacro="http://www.ros.org/wiki/xacro"
        xmlns:ros2_control="http://ros2-control.ros.org/">
-  <xacro:macro name="joint_hardware_interface" params="name initial_pos">
+  <xacro:macro name="arm_hardware_interface" params="name initial_pos">
     <joint name="${name}" type="revolute">
-      <ros2_control name="${name}" type="system">
          <hardware_interface>PositionJointInterface</hardware_interface>
          <command_interface name="position"/>
@@ -16,5 +15,4 @@
            <param name="initial_value">0.0</param>
          </state_interface>
-      </ros2_control>
     </joint>
   </xacro:macro>

Commit message: Point 2h

File: arm_description/urdf/arm.urdf.xacro (robot description, xacro)
@@ -348,8 +348,8 @@
     </inertial>
   </link>
-    <gazebo>
+  <gazebo>
     <plugin filename="ign_ros2_control-system" name="ign_ros2_control::IgnitionROS2ControlPlugin">
-    <parameters>$(find arm_description)/config/arm_joint_controller.yaml</parameters>
-      <controller_manager_prefix_node_name>controller_manager</controller_manager_prefix_node_name>
+    <parameters>$(find arm_control)/config/arm_control.yaml</parameters>
+    <controller_manager_prefix_node_name>controller_manager</controller_manager_prefix_node_name>
     </plugin>
   </gazebo>

File: arm_description/urdf/arm_hardware_interface.xacro (robot description, xacro)
@@ -3,5 +3,5 @@
        xmlns:ros2_control="http://ros2-control.ros.org/">
   <xacro:macro name="arm_hardware_interface" params="name initial_pos">
-    <joint name="${name}" type="revolute">
+      <joint name="${name}" type="revolute">
          <hardware_interface>PositionJointInterface</hardware_interface>
          <command_interface name="position"/>
@@ -15,5 +15,5 @@
            <param name="initial_value">0.0</param>
          </state_interface>
-    </joint>
+      </joint>
   </xacro:macro>
 </robot>

Commit message: beta commit

File: arm_description/urdf/arm.urdf.xacro (robot description, xacro)
@@ -2,4 +2,5 @@
 <robot name="arm" xmlns:xacro="http://www.ros.org/wiki/xacro">
   <xacro:include filename="$(find arm_description)/urdf/arm_hardware_interface.xacro"/>
+  <xacro:include filename="$(find arm_description)/urdf/arm_camera.xacro"/>
   <material name="red">
     <color rgba="1 0 0 1"/>
@@ -347,4 +348,17 @@
       <inertia ixx="6.90013881e-05" ixy="0.0" ixz="0.0" iyy="1.24554875e-04" iyz="0.0" izz="1.04295793e-04"/>
     </inertial>
+  </link>
+  <joint name="camera_joint" type="fixed">
+      <parent link="base_link"/>
+      <child link="camera_link"/>
+      <origin xyz="0 -0.04 0.05" rpy="0 0 -1.57"/>
+  </joint>
+  <link name="camera_link">
+      <visual>
+          <geometry>
+              <box size="0.001 0.003 0.003"/>
+          </geometry>
+          <material name="red"/>
+      </visual>
   </link>
   <gazebo>
@@ -363,3 +377,4 @@
     <xacro:arm_hardware_interface name="j3" initial_pos="0.1" />
   </ros2_control>
+  <xacro:arm_camera name="camera" link_reference="camera_link" />
 </robot>
